File: doc/Layout/strobe.brd (EAGLE design)
At the start: 130 x 90 mm, 20 parts, among them IC1 ATTINY24/44/84-PU, K1 FINDER-30.22, T1 BC337

Commit message: update circuit diagram
Parts:
- removed IRM-05-5: (no value), trafo:VP31
- added U$1: IRM-05-5, meanwell_irm_v5:IRM_05/10
- R2: value wait -> 10k
- R4: value active -> 10k
- moved R6 20.9 mm to (36.8, 39.4)
- moved D1 19.4 mm to (21.6, 39.4)
- moved R1 19.3 mm to (61.0, 47.0)
- moved T1 18.5 mm to (49.5, 47.0)
- moved K1 18.2 mm to (21.6, 53.3)
- moved R3 12.8 mm to (27.9, 34.3), turned to 180 degrees
- moved LED1 12.7 mm to (15.2, 34.3)
- moved S2 11.7 mm to (53.3, 31.8)
- moved R5 7.73 mm to (39.4, 52.1)
- moved LED2 6.48 mm to (35.6, 45.7)
- moved BUZZER 3.81 mm to (6.35, 36.8)
Connections:
- net +5V: no longer IRM-05-5.4
- net GND: now also U$1.V-; no longer IRM-05-5.3
- net N$1: now also U$1.AC/N; no longer IRM-05-5.1
- net N$2: no longer IRM-05-5.2

Commit message: update circuit diagram
Parts:
- IC1: value ATTINY24/44/84-PU -> ATtiny 44A-PU
Changed lines of the file:
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@@
 <element name="C1" library="rcl" package="E2,5-6E" value="100n" x="77.47" y="81.28"/>
 <element name="D1" library="diode" package="DO35-7" value="1N4148" x="21.59" y="39.37"/>
-<element name="IC1" library="attiny24_44_84" package="DIL14" value="ATTINY24/44/84-PU" x="77.47" y="67.31" rot="R270"/>
+<element name="IC1" library="attiny24_44_84" package="DIL14" value="ATtiny 44A-PU" x="77.47" y="67.31" rot="R270"/>
 <element name="JP1" library="pinhead" package="1X06" value="ISP" x="99.06" y="63.5" rot="R270"/>
 <element name="K1" library="relay" package="FINDER-30.22" value="FINDER-30.22" x="21.59" y="53.34" rot="R90">
