File: doc/Layout/strobe.sch (EAGLE design)
At the start: 20 parts, among them IC1 ATTINY24/44/84-PU, K1 FINDER-30.22, T1 BC337

Commit message: update circuit diagram
Parts:
- removed IRM-05-5: (no value), trafo:VP31
- added U$1: IRM-05-5, meanwell_irm_v5:IRM_05/10
- R2: value wait -> 10k
- R4: value active -> 10k
Connections:
- net +5V: no longer IRM-05-5.S4
- net GND: now also U$1.V-; no longer IRM-05-5.S3
- net N$1: now also U$1.AC/N; no longer IRM-05-5.P1
- net N$2: no longer IRM-05-5.P2
Other:
- note added: "blink"
- note added: "wait"
- moved on the sheet: LINE-1, LINE-2
Changed lines of the file:
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@@
 <part name="C1" library="rcl" deviceset="CPOL-EU" device="E2,5-6E" value="100n"/>
 <part name="R1" library="resistor" deviceset="R-EU_" device="0207/10" value="470"/>
-<part name="R2" library="pot" deviceset="TRIM_EU-" device="CA6V" value="wait"/>
+<part name="R2" library="pot" deviceset="TRIM_EU-" device="CA6V" value="10k"/>
 <part name="S1" library="switch-omron" deviceset="10-XX" device="" value="enable"/>
 <part name="LED1" library="led" deviceset="LED" device="3MM" value="enabled"/>
 <part name="T1" library="transistor" deviceset="BC337" device=""/>
 <part name="D1" library="diode" deviceset="1N4148" device="DO35-7" value="1N4148"/>
-<part name="IRM-05-5" library="trafo" deviceset="VP31" device=""/>
 <part name="SUPPLY1" library="supply2" deviceset="+5V" device=""/>
 <part name="GND1" library="supply1" deviceset="GND" device=""/>
@@
 <part name="GND4" library="supply1" deviceset="GND" device=""/>
 <part name="SUPPLY4" library="supply2" deviceset="+5V" device=""/>
-<part name="R4" library="pot" deviceset="TRIM_EU-" device="CA6V" value="active"/>
+<part name="R4" library="pot" deviceset="TRIM_EU-" device="CA6V" value="10k"/>
 <part name="GND5" library="supply1" deviceset="GND" device=""/>
 <part name="S2" library="switch-omron" deviceset="10-XX" device="" value="reset"/>
@@
 <part name="LIGHT" library="con-wago-500" deviceset="W237-102" device=""/>
 <part name="BUZZER" library="con-wago-500" deviceset="W237-102" device=""/>
+<part name="FRAME1" library="frames" deviceset="A4L-LOC" device=""/>
+<part name="U$1" library="meanwell_irm_v5" deviceset="IRM_05/10" device="" value="IRM-05-5"/>
 </parts>
 <sheets>
 <sheet>
 <plain>
+<text x="215.9" y="-5.08" size="1.778" layer="91">blink</text>
+<text x="215.9" y="15.24" size="1.778" layer="91">wait</text>
 </plain>
 <instances>
@@
 <instance part="T1" gate="G$1" x="175.26" y="7.62"/>
 <instance part="D1" gate="G$1" x="210.82" y="27.94" rot="R90"/>
-<instance part="IRM-05-5" gate="1" x="91.44" y="0"/>
-<instance part="SUPPLY1" gate="+5V" x="104.14" y="7.62"/>
+<instance part="SUPPLY1" gate="+5V" x="104.14" y="15.24"/>
 <instance part="GND1" gate="1" x="104.14" y="-10.16"/>
-<instance part="LINE" gate="-1" x="76.2" y="2.54"/>
-<instance part="LINE" gate="-2" x="76.2" y="-2.54"/>
+<instance part="LINE" gate="-1" x="53.34" y="5.08"/>
+<instance part="LINE" gate="-2" x="53.34" y="0"/>
 <instance part="SUPPLY2" gate="+5V" x="66.04" y="58.42"/>
 <instance part="GND2" gate="1" x="66.04" y="35.56"/>
@@
 <instance part="BUZZER" gate="-1" x="231.14" y="83.82" rot="R180"/>
 <instance part="BUZZER" gate="-2" x="231.14" y="78.74" rot="R180"/>
+<instance part="FRAME1" gate="G$1" x="40.64" y="-60.96"/>
+<instance part="U$1" gate="G$1" x="78.74" y="2.54"/>
 </instances>
 <busses>
@@
 <segment>
 <pinref part="LINE" gate="-1" pin="KL"/>
-<pinref part="IRM-05-5" gate="1" pin="P1"/>
-<wire x1="81.28" y1="2.54" x2="81.28" y2="5.08" width="0.1524" layer="91"/>
-<wire x1="81.28" y1="5.08" x2="86.36" y2="5.08" width="0.1524" layer="91"/>
+<wire x1="58.42" y1="5.08" x2="58.42" y2="10.16" width="0.1524" layer="91"/>
+<pinref part="U$1" gate="G$1" pin="AC/N"/>
+<wire x1="58.42" y1="10.16" x2="66.04" y2="10.16" width="0.1524" layer="91"/>
 </segment>
 </net>
@@
 <segment>
 <pinref part="LINE" gate="-2" pin="KL"/>
-<pinref part="IRM-05-5" gate="1" pin="P2"/>
-<wire x1="81.28" y1="-2.54" x2="81.28" y2="-7.62" width="0.1524" layer="91"/>
-<wire x1="81.28" y1="-7.62" x2="86.36" y2="-7.62" width="0.1524" layer="91"/>
+<wire x1="58.42" y1="0" x2="58.42" y2="-5.08" width="0.1524" layer="91"/>
+<wire x1="58.42" y1="-5.08" x2="66.04" y2="-5.08" width="0.1524" layer="91"/>
 </segment>
 </net>
@@
 </segment>
 <segment>
-<pinref part="IRM-05-5" gate="1" pin="S3"/>
 <pinref part="GND1" gate="1" pin="GND"/>
-<wire x1="99.06" y1="-5.08" x2="104.14" y2="-5.08" width="0.1524" layer="91"/>
 <wire x1="104.14" y1="-5.08" x2="104.14" y2="-7.62" width="0.1524" layer="91"/>
+<pinref part="U$1" gate="G$1" pin="V-"/>
+<wire x1="104.14" y1="-5.08" x2="91.44" y2="-5.08" width="0.1524" layer="91"/>
 </segment>
 <segment>
@@
 </segment>
 <segment>
-<pinref part="IRM-05-5" gate="1" pin="S4"/>
 <pinref part="SUPPLY1" gate="+5V" pin="+5V"/>
-<wire x1="99.06" y1="2.54" x2="104.14" y2="2.54" width="0.1524" layer="91"/>
-<wire x1="104.14" y1="2.54" x2="104.14" y2="5.08" width="0.1524" layer="91"/>
+<wire x1="91.44" y1="10.16" x2="104.14" y2="10.16" width="0.1524" layer="91"/>
+<wire x1="104.14" y1="10.16" x2="104.14" y2="12.7" width="0.1524" layer="91"/>
 </segment>
 <segment>

Commit message: update circuit diagram
Parts:
- IC1: value ATTINY24/44/84-PU -> ATtiny 44A-PU
Changed lines of the file:
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@@
 </classes>
 <parts>
-<part name="IC1" library="attiny24_44_84" deviceset="ATTINY24/44/84" device="-PU"/>
+<part name="IC1" library="attiny24_44_84" deviceset="ATTINY24/44/84" device="-PU" value="ATtiny 44A-PU"/>
 <part name="C1" library="rcl" deviceset="CPOL-EU" device="E2,5-6E" value="100n"/>
 <part name="R1" library="resistor" deviceset="R-EU_" device="0207/10" value="470"/>
